Commit message: fix time sleep

File: y1_ros/src/y1_controller/urdf/y10804.urdf (robot description, URDF)
Before this commit: robot y1, 8 links, 7 joints
Links:
- link Link6: mass 0.016469 -> 0.047000

File: y1_ros/src/y1_controller/urdf/y10824_ee.urdf (robot description, URDF)
Before this commit: robot y1, 9 links, 8 joints
Links:
- link Link6: mass  0.479 ->  0.650

Commit message: add master and slave launch

File: y1_ros/src/y1_controller/urdf/y10804.urdf (robot description, URDF)
Before this commit: robot y1, 8 links, 7 joints
Links:
- link Link3: mass 0.84000 -> 0.86000
- link Link4: mass 0.444000 -> 0.464000
- link Link6: mass 0.047000 -> 0.050469

Commit message: fix urdf limit

File: y1_ros/src/y1_controller/urdf/y10804.urdf (robot description, URDF)
Before this commit: robot y1, 8 links, 7 joints
Links:
- link Link3: mass 0.86000 -> 0.84000
- link Link4: mass 0.464000 -> 0.444000
- link Link6: mass 0.050469 -> 0.016469
Joints:
- joint JOINT1: limit lower=-3.0 upper=3.0 effort=30 velocity=5 -> lower=-3.0 upper=3.0 effort=30 velocity=10
- joint JOINT2: limit lower=-3.5 upper=0.2 effort=100 velocity=5 -> lower=-3.5 upper=0.2 effort=120 velocity=10
- joint JOINT3: limit lower=-0.2 upper=4.1 effort=30 velocity=5 -> lower=-0.2 upper=3.5 effort=30 velocity=10
- joint JOINT4: limit lower=-2.5 upper=1.7 effort=10 velocity=20 -> lower=-2.5 upper=1.7 effort=30 velocity=10
- joint JOINT5: limit lower=-2.0 upper=2.0 effort=10 velocity=20 -> lower=-2.0 upper=2.0 effort=20 velocity=30
- joint JOINT6: limit lower=-3.0 upper=3.0 effort=10 velocity=20 -> lower=-3.0 upper=3.0 effort=20 velocity=30

File: y1_ros/src/y1_controller/urdf/y10824_ee.urdf (robot description, URDF)
Before this commit: robot y1, 9 links, 8 joints
Joints:
- joint JOINT1: limit lower=-3.0 upper=3.0 effort=30 velocity=5 -> lower=-3.0 upper=3.0 effort=30 velocity=10
- joint JOINT2: limit lower=-3.5 upper=0.2 effort=100 velocity=5 -> lower=-3.5 upper=0.2 effort=120 velocity=10
- joint JOINT3: limit lower=-0.2 upper=4.1 effort=30 velocity=5 -> lower=-0.2 upper=3.5 effort=30 velocity=10
- joint JOINT4: limit lower=-2.5 upper=1.7 effort=10 velocity=20 -> lower=-2.5 upper=1.7 effort=30 velocity=10
- joint JOINT5: limit lower=-2.0 upper=2.0 effort=10 velocity=20 -> lower=-2.0 upper=2.0 effort=20 velocity=30
- joint JOINT6: limit lower=-3.0 upper=3.0 effort=10 velocity=20 -> lower=-3.0 upper=3.0 effort=20 velocity=30
