Commit message: add mit control mode

File: y1_sdk/example/urdf/y1_with_gripper.urdf (robot description, URDF)
Before this commit: robot y1, 8 links, 7 joints
Links:
- removed link link1
- removed link link2
- removed link link3
- removed link link4
- removed link link5
- removed link link6
- added link Link1, mass 0.893000; collision mesh filename=package://y1_description/meshes/Link1.STL; visual mesh filename=package://y1_description/meshes/Link1.STL
- added link Link2, mass 1.028000; collision mesh filename=package://y1_description/meshes/Link2.STL; visual mesh filename=package://y1_description/meshes/Link2.STL
- added link Link3, mass 0.838; collision mesh filename=package://y1_description/meshes/Link3.STL; visual mesh filename=package://y1_description/meshes/Link3.STL
- added link Link4, mass 0.444000; collision mesh filename=package://y1_description/meshes/Link4.STL; visual mesh filename=package://y1_description/meshes/Link4.STL
- added link Link5, mass 0.363000; collision mesh filename=package://y1_description/meshes/Link5.STL; visual mesh filename=package://y1_description/meshes/Link5.STL
- added link Link6, mass 0.667000; collision mesh filename=package://y1_description/meshes/Link6.STL; visual mesh filename=package://y1_description/meshes/Link6.STL
- link base_link: geometry collision mesh filename=package://y1_description/meshes/base_link.STL; visual mesh filename=package://y1_description/meshes/base_link.STL
Joints:
- removed joint joint1
- removed joint joint2
- removed joint joint3
- removed joint joint4
- removed joint joint5
- removed joint joint6
- added joint JOINT1: type revolute, parent base_link, child Link1, origin xyz=0 0 0.06675 rpy=0 0 0, axis 0 0 -1, limit lower=-3.0 upper=3.0 effort=30 velocity=10
- added joint JOINT2: type revolute, parent Link1, child Link2, origin xyz=0.00075 0 0.055 rpy=1.5708 0 0, axis 0 0 1, limit lower=-3.5 upper=0.2 effort=120 velocity=10
- added joint JOINT3: type revolute, parent Link2, child Link3, origin xyz=-0.28 0 0 rpy=0 0 0, axis 0 0 1, limit lower=-0.2 upper=3.5 effort=30 velocity=10
- added joint JOINT4: type revolute, parent Link3, child Link4, origin xyz=0.215 0.063 0 rpy=0 0 0, axis 0 0 1, limit lower=-2.5 upper=1.7 effort=30 velocity=10
- added joint JOINT5: type revolute, parent Link4, child Link5, origin xyz=0.080817 0.05072 0.00025 rpy=1.5708 0 -0.015918, axis 0 0 1, limit lower=-2.0 upper=2.0 effort=20 velocity=30
- added joint JOINT6: type revolute, parent Link5, child Link6, origin xyz=0.0235 0 0.0440000000000001 rpy=-3.14159265330655 0 0, axis 1 0 0, limit lower=-3.0 upper=3.0 effort=20 velocity=30
