Commit message: fix end pose with urdf.

File: y1_sdk/example/urdf/y1_no_gripper.urdf (robot description, URDF)
Before this commit: robot y1, 9 links, 8 joints
Links:
- removed link gripper_ee
- link Link6: mass  0.650 -> 0.150000; geometry collision mesh filename=package://y1_description/meshes_y1/Link6.STL; visual mesh filename=package://y1_description/meshes_y1/Link6.STL
Joints:
- removed joint Link6_to_gripper_ee
- joint JOINT1: axis 0 0 -1 -> 0 0 1; origin xyz=0 0 0 rpy=0 0 0 -> xyz=0 0 0.06675 rpy=0 0 0
- joint JOINT3: limit lower=-0.2 upper=3.5 effort=30 velocity=10 -> lower=-0.2 upper=3.25 effort=30 velocity=10
- joint JOINT4: limit lower=-2.5 upper=1.7 effort=30 velocity=10 -> lower=-2.35 upper=1.6 effort=30 velocity=10
- joint JOINT5: limit lower=-2.0 upper=2.0 effort=20 velocity=30 -> lower=-1.6 upper=1.6 effort=20 velocity=30
- joint JOINT6: axis 0 0 1 -> 1 0 0; limit lower=-3.0 upper=3.0 effort=20 velocity=30 -> lower=-2.75 upper=2.75 effort=20 velocity=30; origin xyz=0.0235 0 0.044 rpy=3.1416 1.5708 3.1416 -> xyz=0.0235 0 0.0440000000000001 rpy=-3.14159265330655 0 0
- joint fixed_base_joint: axis 0 0 1 -> (none); origin xyz=0 0 0.06675 rpy=0 0 0 -> (none)

File: y1_sdk/example/urdf/y1_with_gripper.urdf (robot description, URDF)
Before this commit: robot y1, 8 links, 7 joints
Links:
- link Link1: geometry collision mesh filename=package://y1_description/meshes/Link1.STL; visual mesh filename=package://y1_description/meshes/Link1.STL
- link Link2: geometry collision mesh filename=package://y1_description/meshes/Link2.STL; visual mesh filename=package://y1_description/meshes/Link2.STL
- link Link3: mass 0.84000 -> 0.838; geometry collision mesh filename=package://y1_description/meshes/Link3.STL; visual mesh filename=package://y1_description/meshes/Link3.STL
- link Link4: geometry collision mesh filename=package://y1_description/meshes/Link4.STL; visual mesh filename=package://y1_description/meshes/Link4.STL
- link Link5: geometry collision mesh filename=package://y1_description/meshes/Link5.STL; visual mesh filename=package://y1_description/meshes/Link5.STL
- link Link6: mass 0.016469 -> 0.667000; geometry collision mesh filename=package://y1_description/meshes/Link6.STL; visual mesh filename=package://y1_description/meshes/Link6.STL
- link base_link: geometry collision mesh filename=package://y1_description/meshes/base_link.STL; visual mesh filename=package://y1_description/meshes/base_link.STL
Joints:
- joint JOINT1: axis 0 0 -1 -> 0 0 1
- joint JOINT3: limit lower=-0.2 upper=3.5 effort=30 velocity=10 -> lower=-0.2 upper=3.25 effort=30 velocity=10
- joint JOINT4: limit lower=-2.5 upper=1.7 effort=30 velocity=10 -> lower=-2.35 upper=1.6 effort=30 velocity=10
- joint JOINT5: limit lower=-2.0 upper=2.0 effort=20 velocity=30 -> lower=-1.6 upper=1.6 effort=20 velocity=30
- joint JOINT6: axis 0 0 1 -> 1 0 0; limit lower=-3.0 upper=3.0 effort=20 velocity=30 -> lower=-2.75 upper=2.75 effort=20 velocity=30; origin xyz=0.0235 0 0.044 rpy=3.1416 1.5708 3.1416 -> xyz=0.0235 0 0.0440000000000001 rpy=-3.14159265330655 0 0
